File: PCB/Rocket/_autosave-Rocket.kicad_sch (KiCad schematic)
At the start: 47 parts, among them J1 Conn_01x08_Pin, J2 Conn_01x04_Pin, J3 Conn_01x07_Pin, J4 Micro_SD_Card, J5 Conn_ARM_JTAG_SWD_10, J6 Conn_01x04_Pin, J7 1987724, SW1 CK_KMS2xxG, SW2 CK_KMS2xxG, U1 STM32L476RGTx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

Commit message: Fixed I2C traces.
Parts:
- J6: footprint Connector_PinSocket_2.54mm:PinSocket_1x04_P2.54mm_Horizontal -> Connector_PinSocket_2.54mm:PinSocket_1x04_P2.54mm_Vertical
Changed lines of the file:
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@@
 			)
 		)
-		(property "Footprint" "Connector_PinSocket_2.54mm:PinSocket_1x04_P2.54mm_Horizontal"
+		(property "Footprint" "Connector_PinSocket_2.54mm:PinSocket_1x04_P2.54mm_Vertical"
 			(at 21.59 57.15 0)
 			(effects
