File: PCB/Rocket/Rocket.kicad_pcb (KiCad board)
At the start: 2 copper layers, 62.7 x 63.5 mm, 49 parts, among them J4 Micro_SD_Card, J5 Conn_ARM_JTAG_SWD_10, J7 1987724, U1 STM32L476RGTx, U2 MIC5365-3.3YC5-TR, U3 MC78L05ACDR2G

Commit message: Updated PCB
Parts:
- added D8: 1N4001, Diode_THT:D_DO-41_SOD81_P10.16mm_Horizontal, F.Cu at (147.5, 32.0)
- added J10: 1987724, 1987724:CONN_1987724_PXC, F.Cu at (161.8, -1.70)
- added J11: 1987724, 1987724:CONN_1987724_PXC, F.Cu at (175.5, 21.8)
- added J2: 1987724, 1987724:CONN_1987724_PXC, F.Cu at (150.0, 21.8)
- added Q1: IRLZ44N, Package_TO_SOT_THT:TO-220-3_Vertical, F.Cu at (162.8, 33.7)
- added R5: 10k, Resistor_SMD:R_0201_0603Metric_Pad0.64x0.40mm_HandSolder, F.Cu at (172.5, 30.8)
- added R6: 220, Resistor_SMD:R_0201_0603Metric_Pad0.64x0.40mm_HandSolder, F.Cu at (172.5, 32.5)
